File: hardware/pir-night-light/pir-night-light.kicad_sch (KiCad schematic)
At the start: 15 parts, among them J1 PIR Sensor, Q1 2N3904, U1 ATtiny85-20P

Commit message: Added pullup resistor on MCU reset pin
Parts:
- added R8: 10k, symbol Device:R
Connections:
- net +BATT: now also R8.2
- net at U1.1 (~{RESET}/PB5): now also R8.1
Changed lines of the file:
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@@
     (pin "2")
+  )
+  (symbol (lib_id "power:+BATT") (at 154.94 123.19 270) (unit 1)
+    (in_bom yes) (on_board yes) (fields_autoplaced)
+    (property "Reference" "#PWR010" (id 0) (at 151.13 123.19 0)
+      (effects (font (size 1.27 1.27)) hide)
+    )
+    (property "Value" "+BATT" (id 1) (at 158.115 123.1899 90)
+      (effects (font (size 1.27 1.27)) (justify left))
+    )
+    (property "Footprint" "" (id 2) (at 154.94 123.19 0)
+      (effects (font (size 1.27 1.27)) hide)
+    )
+    (property "Datasheet" "" (id 3) (at 154.94 123.19 0)
+      (effects (font (size 1.27 1.27)) hide)
+    )
+    (pin "1")
   )
   (symbol (lib_id "power:Earth") (at 92.71 55.88 0) (unit 1)
@@
     (pin "2")
   )
+  (symbol (lib_id "Device:R") (at 151.13 123.19 90) (unit 1)
+    (in_bom yes) (on_board yes)
+    (property "Reference" "R8" (id 0) (at 151.13 125.73 90))
+    (property "Value" "10k" (id 1) (at 151.13 123.19 90))
+    (property "Footprint" "" (id 2) (at 151.13 124.968 90)
+      (effects (font (size 1.27 1.27)) hide)
+    )
+    (property "Datasheet" "~" (id 3) (at 151.13 123.19 0)
+      (effects (font (size 1.27 1.27)) hide)
+    )
+    (pin "1")
+    (pin "2")
+  )
   (symbol (lib_id "power:Earth") (at 184.15 118.11 0) (unit 1)
     (in_bom yes) (on_board yes) (fields_autoplaced)
@@
       (reference "#PWR09") (unit 1) (value "Earth") (footprint "")
     )
+    (path "/318cca53-4454-429e-b3f4-efb5d4ce3eeb"
+      (reference "#PWR010") (unit 1) (value "+BATT") (footprint "")
+    )
     (path "/252b166a-0097-4642-8cbf-ec7dd6976b10"
       (reference "D1") (unit 1) (value "RED LED") (footprint "")
@@
       (reference "R7") (unit 1) (value "100R") (footprint "")
     )
+    (path "/cd5c661e-5955-464f-9c17-e3855a0a3a02"
+      (reference "R8") (unit 1) (value "10k") (footprint "")
+    )
     (path "/42792f24-8f19-4181-b703-2e87c0193377"

Commit message: Schematic updated to support low battery level warning
Parts:
- added R10: 1k, symbol Device:R
- added R9: 10k, symbol Device:R
Connections:
- net Earth: now also R10.2
- net LED_CONTROL: now also R9.1
- net LDR_DIVIDER renamed ADC
- net ADC: now also R10.1, R9.2
Other:
- note added: "Approx. 21mA"
- note added: "Battery Level Measurement"
- moved on the sheet: R1, R2
